File: kicad/sbrb/sbrb.kicad_pcb (KiCad board)
At the start: 2 copper layers, 6 parts, among them J1 Conn_Batt, J2 Motor1, J3 Motor2, U1 XIAO-ESP32-S3-DIP, U2 MINI-360

Commit message: Initial schematic
Parts:
- added C3: 0.1uF, Capacitor_SMD:C_0805_2012Metric, F.Cu at (209.2, 68.5)
- added C4: 0.1uF, Capacitor_SMD:C_0805_2012Metric, F.Cu at (200.5, 68.3)
- added J4: motor1_sense, Connector_JST:JST_XH_B4B-XH-AM_1x04_P2.50mm_Vertical, F.Cu at (149.2, 88.7)
- added J5: motor2_sense, Connector_JST:JST_XH_B4B-XH-AM_1x04_P2.50mm_Vertical, F.Cu at (139.6, 88.7)
- added R1: 32k, Resistor_SMD:R_0805_2012Metric, F.Cu at (168.6, 57.2)
- added R2: 10k, Resistor_SMD:R_0805_2012Metric, F.Cu at (173.6, 57.0)
- added U3: SparkFun_TB6612FNG, jaguilar:TB6612FNG_Breakout, F.Cu at (98.2, 75.9)
- U1: value XIAO-ESP32-S3-DIP -> ESP32-S3-Zero; footprint RF_Module:MCU_Seeed_ESP32C3 -> jaguilar:ESP32-S3-Zero_Breakout
- U2: footprint mini360:mini360 -> jaguilar:mini360
- moved U1 77.1 mm to (141.3, 59.9), turned to 90 degrees
- moved U2 33.5 mm to (95.1, 54.5)
- moved J2 28.4 mm to (102.2, 90.3), turned to 180 degrees
- moved J1 27.2 mm to (116.5, 46.4)
- moved C1 20.5 mm to (108.6, 48.5), turned to -90 degrees
- moved J3 17.4 mm to (90.0, 89.3)
Connections:
- U1 pad 1: unconnected-(U1-GPIO1/D0/A0-Pad1) -> 5V
- U1 pad 11: unconnected-(U1-GPIO9/D10/A10/MOSI-Pad11) -> /pwmb
- U1 pad 12: 3V3 -> /bin2
- U1 pad 13: GND -> /bin1
- U1 pad 14: 5V -> /ain1
- U1 pad 15: (no net) -> /ain2
- U1 pad 16: (no net) -> /pwma
- U1 pad 17: (no net) -> unconnected-(U1-TX/IO43-Pad17)
- U1 pad 18: (no net) -> unconnected-(U1-RX/IO44-Pad18)
- U1 pad 2: unconnected-(U1-GPIO2/DA/A1-Pad2) -> GND
- U1 pad 3: unconnected-(U1-GPIO3/D2/A2-Pad3) -> 3V3
- U1 pad 4: unconnected-(U1-GPIO4/D3/A3-Pad4) -> /batt_prot
- U1 pad 5: unconnected-(U1-GPIO5/D4/I2C_SDA-Pad5) -> Net-(J4-Pin_2)
- U1 pad 6: unconnected-(U1-GPIO9/D5/I2C_SCL-Pad6) -> Net-(J4-Pin_3)
- U1 pad 7: unconnected-(U1-U0TXD/D6/TX-Pad7) -> Net-(J5-Pin_2)
- U1 pad 8: unconnected-(U1-U0RXD/D7/RX-Pad8) -> Net-(J5-Pin_3)
Routing:
- net GND: track 0.00 -> 121.9 mm
- net VBATT: track 0.00 -> 58.5 mm
- net Net-(J2-Pin_2): track 0.00 -> 13.4 mm
- net Net-(J2-Pin_1): track 0.00 -> 12.3 mm
- net Net-(J3-Pin_1): track 0.00 -> 11.0 mm
- net Net-(J3-Pin_2): track 0.00 -> 10.1 mm
- net 5V: track 0.00 -> 8.99 mm

Commit message: Finishe design
Parts:
- added C2: 470uF, Capacitor_THT:CP_Radial_D8.0mm_P3.80mm, F.Cu at (111.8, 72.4)
- added F1: 3A, Fuse:Fuse_Schurter_UMT250, F.Cu at (114.7, 51.8)
- added R3: 2.2k, Resistor_SMD:R_0805_2012Metric, F.Cu at (122.5, 74.4)
- added R4: 2.2k, Resistor_SMD:R_0805_2012Metric, F.Cu at (125.2, 74.4)
- added SW1: SW_Push, Button_Switch_SMD:SW_SPST_FSMSM, F.Cu at (121.5, 60.5)
- added U4: GY-521_MPU6050, jaguilar:GY-521, F.Cu at (121.5, 85.5)
- C1: footprint Capacitor_THT:CP_Axial_L11.0mm_D8.0mm_P15.00mm_Horizontal -> Capacitor_THT:CP_Radial_D6.3mm_P2.50mm
- moved C3 111.0 mm to (99.2, 83.5)
- moved C4 111.0 mm to (90.5, 83.3), turned to 180 degrees
- moved R2 51.5 mm to (123.6, 69.5)
- moved R1 45.6 mm to (123.6, 64.7)
- moved J4 10.0 mm to (139.2, 88.6)
- moved J5 10.0 mm to (149.6, 88.6)
- moved J1 5.59 mm to (121.5, 48.9)
- moved U3 5.59 mm to (95.7, 70.9)
- moved C1 2.86 mm to (107.2, 51.0)
- moved J3 2.71 mm to (92.5, 90.3), turned to 180 degrees
- moved U2 2.50 mm to (95.2, 52.0)
Connections:
- J1 pad 1: VBATT -> /VBATT_CONN_TO_SW
- U1 pad 10: unconnected-(U1-IO7-Pad10) -> /SDA
- U1 pad 9: unconnected-(U1-IO6-Pad9) -> /SCL
Routing:
- net 3V3: track 0.00 -> 95.6 mm
- net /pwmb: track 0.00 -> 67.0 mm
- net GND: track 121.9 -> 183.8 mm
- net /bin2: track 0.00 -> 61.6 mm
- net /bin1: track 0.00 -> 56.2 mm
- net /SDA: track 0.00 -> 48.5 mm
- net /ain1: track 0.00 -> 48.3 mm
- net /ain2: track 0.00 -> 42.9 mm
- net /SCL: track 0.00 -> 39.6 mm
- net /pwma: track 0.00 -> 36.7 mm
- net 5V: track 8.99 -> 41.6 mm, vias 0 -> 2
- net Net-(J4-Pin_2): track 0.00 -> 19.2 mm
- net /batt_prot: track 0.00 -> 18.7 mm, vias 0 -> 1
- net Net-(J5-Pin_2): track 0.00 -> 18.6 mm
- net VBATT: track 58.5 -> 76.3 mm, vias 0 -> 2
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Other:
- board outline added: 70 x 50 mm
- copper layers 2 -> 4
