File: kicad/sbrb/sbrb.kicad_sch (KiCad schematic)
At the start: 10 parts, among them J1 Conn_Batt, J2 Motor1, J3 Motor2, U1 XIAO-ESP32-S3-DIP, U2 MINI-360, U3 SparkFun_TB6612FNG

Commit message: Initial schematic
Parts:
- added J4: motor1_sense, Connector_JST:JST_XH_B4B-XH-AM_1x04_P2.50mm_Vertical, symbol Connector_Generic:Conn_01x04
- added J5: motor2_sense, Connector_JST:JST_XH_B4B-XH-AM_1x04_P2.50mm_Vertical, symbol Connector_Generic:Conn_01x04
- added R1: 32k, Resistor_SMD:R_0805_2012Metric, symbol Device:R
- added R2: 10k, Resistor_SMD:R_0805_2012Metric, symbol Device:R
- C3, C4: footprint (none) -> Capacitor_SMD:C_0805_2012Metric
- U1: value XIAO-ESP32-S3-DIP -> ESP32-S3-Zero; footprint RF_Module:MCU_Seeed_ESP32C3 -> jaguilar:ESP32-S3-Zero_Breakout; symbol Seeed_Studio_XIAO_Series:XIAO-ESP32-S3-DIP -> jaguilar:Waveshare_ESP32_S3_Zero
- U2: footprint mini360:mini360 -> jaguilar:mini360; symbol mini360:MINI-360_Buck_Converter -> jaguilar:MINI-360_Buck_Converter
- U3: footprint SparkFun_TB6612FNG:TB6612FNG_Breakout -> jaguilar:TB6612FNG_Breakout; symbol APrkFun_TB6612FNG:SparkFun_TB6612FNG -> jaguilar:SparkFun_TB6612FNG
Connections:
- net 3V3: now also U1.3 (3V3), U3.15 (VCC), U3.4 (STBY), J4.4 (Pin_4), J5.4 (Pin_4); no longer U1.12 (VCC_3V3)
- net 5V: now also U1.1 (5V); no longer U1.14 (VBUS), U3.15 (VCC)
- net GND: now also U1.2 (GND), J4.1 (Pin_1), J5.1 (Pin_1), R2.2; no longer U1.13 (GND)
- net VBATT: now also R1.1
- net pwma: now reaches U3.1 (PWMA)
- net pwma: now also U1.16 (IO13)
- net ain2: now reaches U3.2 (AIN2)
- net ain2: now also U1.15 (IO12)
- net ain1: now reaches U3.3 (AIN1)
- net ain1: now also U1.14 (IO11)
- net bin1: now reaches U3.5 (BIN1)
- net bin1: now also U1.13 (IO10)
- net bin2: now reaches U3.6 (BIN2)
- net bin2: now also U1.12 (IO9)
- net pwmb: now reaches U3.7 (PWMB)
- net pwmb: now also U1.11 (IO8)
- net batt_prot: now reaches U1.4 (IO1)
- net batt_prot: now also R1.2, R2.1
- net at U1.5 (IO2): now also J4.2 (Pin_2)
- net at U1.6 (IO3): now also J4.3 (Pin_3)
- net at U1.7 (IO4): now also J5.2 (Pin_2)
- net at U1.8 (IO5): now also J5.3 (Pin_3)

Commit message: Finishe design
Parts:
- added F1: 3A, Fuse:Fuse_Schurter_UMT250, symbol Device:Fuse
- added R3, R4: 2.2k, Resistor_SMD:R_0805_2012Metric, symbol Device:R
- added SW1: SW_Push, Button_Switch_SMD:SW_SPST_FSMSM, symbol Switch:SW_Push
- added U4: GY-521_MPU6050, jaguilar:GY-521, symbol jaguilar:GY-521_MPU6050
- C1: footprint Capacitor_THT:CP_Axial_L11.0mm_D8.0mm_P15.00mm_Horizontal -> Capacitor_THT:CP_Radial_D6.3mm_P2.50mm
- C2: footprint (none) -> Capacitor_THT:CP_Radial_D8.0mm_P3.80mm
Connections:
- net 3V3: now also R3.1, R4.1, U4.1 (VCC)
- net GND: now also U4.2 (GND)
- net VBATT: now also F1.1; no longer J1.1 (Pin_1)
- net SDA: now reaches U1.10 (IO7)
- net SDA: now also R3.2, U4.4 (SDA)
- net SCL: now reaches U1.9 (IO6)
- net SCL: now also R4.2, U4.3 (SCL)
- new net VBATT_CONN_TO_SW: J1.1 (Pin_1), SW1.1
- new net VBATT_SW_TO_FUSE: F1.2, SW1.2
- no-connect marks 0 -> 6
Other:
- moved on the sheet: J1

Commit message: Add needed diode.
Parts:
- added D1: 1N5819, Diode_THT:D_DO-41_SOD81_P10.16mm_Horizontal, symbol Diode:1N5819
Connections:
- net 5V: now also D1.2 (A); no longer U1.1 (5V)
- new net: D1.1 (K), U1.1 (5V)
Changed lines of the file:
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@@
+	(wire
+		(pts
+			(xy 68.58 40.64) (xy 67.31 40.64)
+		)
+		(stroke
+			(width 0)
+			(type default)
+		)
+	)
 	(wire
 		(pts
@@
 	(wire
 		(pts
-			(xy 78.74 40.64) (xy 67.31 40.64)
+			(xy 78.74 40.64) (xy 76.2 40.64)
 		)
 		(stroke
@@
 					(unit 1)
 				)
+			)
+		)
+	)
+	(symbol
+		(lib_id "Diode:1N5819")
+		(at 72.39 40.64 180)
+		(unit 1)
+		(body_style 1)
+		(exclude_from_sim no)
+		(in_bom yes)
+		(on_board yes)
+		(in_pos_files yes)
+		(dnp no)
+		(fields_autoplaced yes)
+		(property "Reference" "D1"
+			(at 72.7075 34.29 0)
+			(show_name no)
+			(do_not_autoplace no)
+			(effects
+				(font
+					(size 1.27 1.27)
+				)
+			)
+		)
+		(property "Value" "1N5819"
+			(at 72.7075 36.83 0)
+			(show_name no)
+			(do_not_autoplace no)
+			(effects
+				(font
+					(size 1.27 1.27)
+				)
+			)
+		)
+		(property "Footprint" "Diode_THT:D_DO-41_SOD81_P10.16mm_Horizontal"
+			(at 72.39 36.195 0)
+			(hide yes)
+			(show_name no)
+			(do_not_autoplace no)
+			(effects
+				(font
+					(size 1.27 1.27)
+				)
+			)
+		)
+		(property "Datasheet" "http://www.vishay.com/docs/88525/1n5817.pdf"
+			(at 72.39 40.64 0)
+			(hide yes)
+			(show_name no)
+			(do_not_autoplace no)
+			(effects
+				(font
+					(size 1.27 1.27)
+				)
+			)
+		)
+		(property "Description" "40V 1A Schottky Barrier Rectifier Diode, DO-41"
+			(at 72.39 40.64 0)
+			(hide yes)
+			(show_name no)
+			(do_not_autoplace no)
+			(effects
+				(font
+					(size 1.27 1.27)
+				)
+			)
+		)
+		(pin "1"
+		)
+		(pin "2"
+		)
+		(instances
+			(project ""
+				(path "/3edb316a-46d5-4aff-aa24-301c1d17e106"
+					(reference "D1")
+					(unit 1)
+				)
